File: OW_PDB.kicad_pcb (KiCad board)
At the start: 2 copper layers, 68.6 x 42.2 mm, 9 parts, among them J1 XT60 VESC, J2 XT60 Main Battery, J3 XT60 Expansion Cell, J4 XT30 XLite Battery, J5 HDMI Balance, J6 JST-PH XLite Balance C13-24, J7 JST-PH XLite Balance C0-12

Commit message: Make connections closer on PCB
Parts:
- moved J6 28.7 mm to (115.0, 96.0)
- moved J1 24.4 mm to (134.6, 82.4)
- moved J4 22.0 mm to (124.9, 67.5)
- moved F2 17.2 mm to (115.8, 73.2)
- moved F1 16.5 mm to (115.8, 82.3)
- moved J3 14.4 mm to (106.3, 67.5)
- moved J2 4.93 mm to (106.2, 82.5)
- moved J7 4.86 mm to (114.0, 103.6)
- moved J5 4.36 mm to (102.0, 97.3)
Routing:
- net Net-(BT1--): track 0.00 -> 29.7 mm
- net Net-(J5-Pin_11): track 37.3 -> 8.42 mm
- net Net-(J5-Pin_18): track 52.7 -> 24.2 mm
- net Net-(J5-Pin_17): track 50.5 -> 22.0 mm
- net Net-(J5-Pin_16): track 48.3 -> 19.9 mm
- net Net-(J5-Pin_15): track 46.1 -> 17.7 mm
- net Net-(J5-Pin_14): track 43.9 -> 15.5 mm
- net Net-(J5-Pin_13): track 41.7 -> 13.4 mm
- net Net-(J5-Pin_12): track 39.5 -> 11.2 mm
- net Net-(J1-Pin_2): track 21.5 -> 13.3 mm
- net Net-(BT1-+): track 42.8 -> 34.6 mm
- net Net-(J5-Pin_9): track 24.9 -> 27.3 mm
- net Net-(J5-Pin_10): track 31.1 -> 33.5 mm
- net Net-(J5-Pin_8): track 22.7 -> 25.1 mm
- net Net-(J5-Pin_7): track 20.5 -> 22.9 mm
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Other:
- board size 68.6 x 42.2 mm -> 43.7 x 48.8 mm
- board text removed: "C0"
